File: hardware/kicad/RunicMesh.kicad_pcb (KiCad board)
At the start: 2 copper layers, 0 parts

Commit message: updates to the schematic
Parts:
- added Battery1: 18650, Battery:BatteryHolder_Keystone_1042_1x18650, F.Cu at (149.2, 98.5)
- added C2: 10µF, Capacitor_SMD:CP_Elec_3x5.3, F.Cu at (108.2, 112.3)
- added C3: 10µF, Capacitor_SMD:CP_Elec_3x5.3, F.Cu at (108.2, 117.1)
- added C4: 0.1µF, Capacitor_SMD:CP_Elec_3x5.3, F.Cu at (108.2, 122.0)
- added LED1: G, LED_SMD:LED_0201_0603Metric_Pad0.64x0.40mm_HandSolder, F.Cu at (125.7, 117.3)
- added LED2: R, LED_SMD:LED_0201_0603Metric_Pad0.64x0.40mm_HandSolder, F.Cu at (125.7, 119.1)
- added Q1: IRLML6244, Package_TO_SOT_SMD:SOT-23, F.Cu at (116.5, 112.3)
- added Q2: IRLML6244, Package_TO_SOT_SMD:SOT-23, F.Cu at (116.5, 116.9)
- added R1: 1k, Resistor_SMD:R_0201_0603Metric, F.Cu at (112.8, 110.7)
- added R2: 1k, Resistor_SMD:R_0201_0603Metric, F.Cu at (112.8, 112.5)
- added R3: 0.4, Resistor_SMD:R_0201_0603Metric, F.Cu at (112.8, 114.2)
- added Rprog1: 1.2K, Resistor_SMD:R_0201_0603Metric, F.Cu at (112.8, 116.0)
- added Rprog2: 1K, Resistor_SMD:R_0201_0603Metric, F.Cu at (112.8, 117.7)
- added Rprog3: 100, Resistor_SMD:R_0201_0603Metric, F.Cu at (112.8, 119.5)
- added U1: TP4056-42-ESOP8, Package_SO:SOIC-8-1EP_3.9x4.9mm_P1.27mm_EP2.41x3.3mm_ThermalVias, F.Cu at (123.2, 113.2)
- added U2: DW01A, Package_TO_SOT_SMD:SOT-23-6, F.Cu at (121.5, 118.8)
