File: hardware/kicad/RunicMesh.kicad_sch (KiCad schematic)
At the start: 7 parts, among them U1 TP4056-42-ESOP8

Commit message: Change power/charging circuit to have LED for chargin status
Parts:
- removed status1: LED, LED_SMD:LED-L1T2_LUMILEDS, symbol Device:LED
- added LED1: G, symbol Device:LED
- added LED2: R, symbol Device:LED
- added R1, R2: 1k, symbol Device:R
- R3: value 10k -> 0.4; footprint Resistor_SMD:R_0201_0603Metric -> (none)
- Rprog1: renamed from R4; value Rprog -> 1.2K
Connections:
- net +5V: now also R3.2; no longer C2.1, U1.8 (CE)
- net GND: no longer U1.6 (~{STDBY})
- net at U1.7 (~{CHRG}): now also R1.2; no longer R3.2
- net at R3.1: now also C2.1, U1.8 (CE), LED1.2 (A), LED2.2 (A)
- new net: LED1.1 (K), R2.1
- new net: R2.2, U1.6 (~{STDBY})
- new net: LED2.1 (K), R1.1
Other:
- moved on the sheet: Battery1, U1

Commit message: Update power part with overdischarge and overcharge protections
Parts:
- added Q1, Q2: IRLML6244, Package_TO_SOT_SMD:SOT-23, symbol Transistor_FET:IRLML6244
- added Rprog2: 1K, Resistor_SMD:R_0201_0603Metric, symbol Device:R
- added U2: DW01A, Package_TO_SOT_SMD:SOT-23-6, symbol Battery_Management:DW01A
- LED1, LED2: footprint (none) -> LED_SMD:LED_0201_0603Metric_Pad0.64x0.40mm_HandSolder
- R1, R2, R3: footprint (none) -> Resistor_SMD:R_0201_0603Metric
Connections:
- net GND: now also Q1.2 (S), U2.6 (GND)
- net B+: now reaches Battery1.1 (+), C3.1, U1.5 (BAT)
- net B+: now also U2.5 (VCC)
- net at C2.1, R3.1, U1.8 (CE): now also LED1.1 (K), LED2.1 (K); no longer LED1.2 (A), LED2.2 (A)
- net at R2.1: now also LED1.2 (A); no longer LED1.1 (K)
- net at R1.1: now also LED2.2 (A); no longer LED2.1 (K)
- new net: Q2.1 (G), U2.3 (OC)
- new net: Q1.3 (D), Q2.2 (S)
- new net: Rprog2.2, U2.2 (CS)
- new net: Q1.1 (G), U2.1 (OD)
- new net B-: Q2.3 (D), Rprog2.1

Commit message: Update power part with overdischarge and overcharge protections
Parts:
- added C4: 0.1µF, Capacitor_SMD:CP_Elec_3x5.3, symbol Device:C_Polarized
- added Rprog3: 100, Resistor_SMD:R_0201_0603Metric, symbol Device:R
Connections:
- net B+: now also Rprog3.2; no longer U2.5 (VCC)
- net GND: now also C4.2
- net at Q2.1 (G), U2.3 (OC): now also Q1.1 (G), U2.1 (OD)
- new net: C4.1, Rprog3.1, U2.5 (VCC)
Other:
- moved on the sheet: U2
Changed lines of the file:
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@@
+	)
+	(junction
+		(at 104.14 33.02)
+		(diameter 0)
+		(color 0 0 0 0)
 	)
 	(junction
@@
 	)
 	(junction
-		(at 121.92 54.61)
-		(diameter 0)
-		(color 0 0 0 0)
-	)
-	(junction
 		(at 88.9 33.02)
 		(diameter 0)
@@
 	)
 	(junction
+		(at 104.14 40.64)
+		(diameter 0)
+		(color 0 0 0 0)
+	)
+	(junction
 		(at 59.69 25.4)
 		(diameter 0)
@@
 		(color 0 0 0 0)
 	)
+	(junction
+		(at 114.3 46.99)
+		(diameter 0)
+		(color 0 0 0 0)
+	)
 	(wire
 		(pts
@@
 	(wire
 		(pts
+			(xy 104.14 33.02) (xy 106.68 33.02)
+		)
+		(stroke
+			(width 0)
+			(type default)
+		)
+	)
+	(wire
+		(pts
 			(xy 38.1 38.1) (xy 38.1 55.88)
 		)
@@
 	(wire
 		(pts
-			(xy 96.52 46.99) (xy 109.22 46.99)
+			(xy 96.52 46.99) (xy 114.3 46.99)
 		)
 		(stroke
@@
 	(wire
 		(pts
-			(xy 88.9 33.02) (xy 101.6 33.02)
+			(xy 104.14 40.64) (xy 88.9 40.64)
+		)
+		(stroke
+			(width 0)
+			(type default)
+		)
+	)
+	(wire
+		(pts
+			(xy 88.9 33.02) (xy 93.98 33.02)
 		)
 		(stroke
@@
 	(wire
 		(pts
+			(xy 101.6 33.02) (xy 104.14 33.02)
+		)
+		(stroke
+			(width 0)
+			(type default)
+		)
+	)
+	(wire
+		(pts
 			(xy 49.53 38.1) (xy 38.1 38.1)
 		)
@@
 	(wire
 		(pts
-			(xy 109.22 46.99) (xy 109.22 43.18)
-		)
-		(stroke
-			(width 0)
-			(type default)
-		)
-	)
-	(wire
-		(pts
-			(xy 114.3 43.18) (xy 114.3 46.99)
+			(xy 114.3 46.99) (xy 114.3 43.18)
+		)
+		(stroke
+			(width 0)
+			(type default)
+		)
+	)
+	(wire
+		(pts
+			(xy 119.38 43.18) (xy 119.38 46.99)
+		)
+		(stroke
+			(width 0)
+			(type default)
+		)
+	)
+	(wire
+		(pts
+			(xy 119.38 46.99) (xy 114.3 46.99)
 		)
 		(stroke
@@
 	(wire
 		(pts
-			(xy 101.6 38.1) (xy 101.6 40.64)
+			(xy 106.68 38.1) (xy 106.68 40.64)
 		)
 		(stroke
@@
 	(wire
 		(pts
-			(xy 121.92 50.8) (xy 121.92 54.61)
+			(xy 127 50.8) (xy 127 54.61)
 		)
 		(stroke
@@
 	(wire
 		(pts
-			(xy 101.6 40.64) (xy 88.9 40.64)
-		)
-		(stroke
-			(width 0)
-			(type default)
-		)
-	)
-	(wire
-		(pts
-			(xy 121.92 54.61) (xy 119.38 54.61)
+			(xy 106.68 40.64) (xy 104.14 40.64)
+		)
+		(stroke
+			(width 0)
+			(type default)
+		)
+	)
+	(wire
+		(pts
+			(xy 119.38 54.61) (xy 127 54.61)
 		)
 		(stroke
@@
 	(wire
 		(pts
-			(xy 127 54.61) (xy 121.92 54.61)
-		)
-		(stroke
-			(width 0)
-			(type default)
-		)
-	)
-	(wire
-		(pts
-			(xy 121.92 38.1) (xy 121.92 43.18)
+			(xy 127 38.1) (xy 127 43.18)
 		)
 		(stroke
@@
 	)
 	(symbol
+		(lib_id "Device:R")
+		(at 97.79 33.02 270)
+		(unit 1)
+		(exclude_from_sim no)
+		(in_bom yes)
+		(on_board yes)
+		(dnp no)
+		(fields_autoplaced yes)
+		(property "Reference" "Rprog3"
+			(at 97.79 39.37 90)
+			(effects
+				(font
+					(size 1.27 1.27)
+				)
+				(hide yes)
+			)
+		)
+		(property "Value" "100"
+			(at 97.79 29.21 90)
+			(effects
+				(font
+					(size 1.27 1.27)
+				)
+			)
+		)
+		(property "Footprint" "Resistor_SMD:R_0201_0603Metric"
+			(at 97.79 31.242 90)
+			(effects
+				(font
+					(size 1.27 1.27)
+				)
+				(hide yes)
+			)
+		)
+		(property "Datasheet" "~"
+			(at 97.79 33.02 0)
+			(effects
+				(font
+					(size 1.27 1.27)
+				)
+				(hide yes)
+			)
+		)
+		(property "Description" "Resistor"
+			(at 97.79 33.02 0)
+			(effects
+				(font
+					(size 1.27 1.27)
+				)
+				(hide yes)
+			)
+		)
+		(pin "1"
+		)
+		(pin "2"
+		)
+		(instances
+			(project "RunicMesh"
+				(path "/845d8e1e-718e-4ec4-be16-16f250b95f5e"
+					(reference "Rprog3")
+					(unit 1)
+				)
+			)
+		)
+	)
+	(symbol
 		(lib_id "Device:C_Polarized")
 		(at 77.47 36.83 0)
@@
 	(symbol
 		(lib_id "Device:R")
-		(at 121.92 46.99 180)
+		(at 127 46.99 180)
 		(unit 1)
 		(exclude_from_sim no)
@@
 		(fields_autoplaced yes)
 		(property "Reference" "Rprog2"
-			(at 115.57 46.99 90)
+			(at 120.65 46.99 90)
 			(effects
 				(font
@@
 		)
 		(property "Value" "1K"
-			(at 124.46 46.9899 0)
+			(at 129.54 46.9899 0)
 			(effects
 				(font
@@
 		)
 		(property "Footprint" "Resistor_SMD:R_0201_0603Metric"
-			(at 123.698 46.99 90)
+			(at 128.778 46.99 90)
 			(effects
 				(font
@@
 		)
 		(property "Datasheet" "~"
-			(at 121.92 46.99 0)
+			(at 127 46.99 0)
 			(effects
 				(font
@@
 		)
 		(property "Description" "Resistor"
-			(at 121.92 46.99 0)
+			(at 127 46.99 0)
 			(effects
 				(font
@@
 	)
 	(symbol
-		(lib_id "Battery_Management:DW01A")
-		(at 111.76 35.56 0)
+		(lib_id "Device:C_Polarized")
+		(at 104.14 36.83 0)
 		(unit 1)
 		(exclude_from_sim no)
@@
 		(dnp no)
 		(fields_autoplaced yes)
+		(property "Reference" "C4"
+			(at 107.95 34.6709 0)
+			(effects
+				(font
+					(size 1.27 1.27)
+				)
+				(justify left)
+				(hide yes)
+			)
+		)
+		(property "Value" "0.1µF"
+			(at 107.95 37.2109 0)
+			(effects
+				(font
+					(size 1.27 1.27)
+				)
+				(justify left)
+			)
+		)
+		(property "Footprint" "Capacitor_SMD:CP_Elec_3x5.3"
+			(at 105.1052 40.64 0)
+			(effects
+				(font
+					(size 1.27 1.27)
+				)
+				(hide yes)
+			)
+		)
+		(property "Datasheet" "~"
+			(at 104.14 36.83 0)
+			(effects
+				(font
+					(size 1.27 1.27)
+				)
+				(hide yes)
+			)
+		)
+		(property "Description" "Polarized capacitor"
+			(at 104.14 36.83 0)
+			(effects
+				(font
+					(size 1.27 1.27)
+				)
+				(hide yes)
+			)
+		)
+		(pin "1"
+		)
+		(pin "2"
+		)
+		(instances
+			(project "RunicMesh"
+				(path "/845d8e1e-718e-4ec4-be16-16f250b95f5e"
+					(reference "C4")
+					(unit 1)
+				)
+			)
+		)
+	)
+	(symbol
+		(lib_id "Battery_Management:DW01A")
+		(at 116.84 35.56 0)
+		(unit 1)
+		(exclude_from_sim no)
+		(in_bom yes)
+		(on_board yes)
+		(dnp no)
+		(fields_autoplaced yes)
 		(property "Reference" "U2"
-			(at 111.76 25.4 0)
+			(at 116.84 25.4 0)
 			(effects
 				(font
@@
 		)
 		(property "Value" "DW01A"
-			(at 111.76 27.94 0)
+			(at 116.84 27.94 0)
 			(effects
 				(font
@@
 		)
 		(property "Footprint" "Package_TO_SOT_SMD:SOT-23-6"
-			(at 111.76 35.56 0)
+			(at 116.84 35.56 0)
 			(effects
 				(font
@@
 		)
 		(property "Datasheet" "https://hmsemi.com/downfile/DW01A.PDF"
-			(at 111.76 35.56 0)
+			(at 116.84 35.56 0)
 			(effects
 				(font
@@
 		)
 		(property "Description" "Overcharge, overcurrent and overdischarge protection IC for single cell lithium-ion/polymer battery"
-			(at 112.014 34.036 0)
-			(effects
-				(font
+			(at 117.094 34.036 0)
+			(effects
+				(font

Commit message: updates to the schematic
Parts:
- added D1, D3: D, Diode_SMD:D_0201_0603Metric, symbol Device:D
- added D2: D, symbol Device:D
- added J1: USB_C_Receptacle, Connector_USB:USB_C_Receptacle_Amphenol_12401548E4-2A, symbol Connector:USB_C_Receptacle
- added R4: 5.1k, Resistor_SMD:R_0201_0603Metric, symbol Device:R
Connections:
- net +5V: now also D1.1 (K)
- net GND: now also Q2.2 (S), Rprog2.1, D2.1 (K), D3.1 (K), J1.A1 (GND), J1.A12 (GND), J1.B1 (GND), J1.B12 (GND), R4.2
- net at Q2.1 (G), U2.3 (OC): no longer Q1.1 (G), U2.1 (OD)
- net at Q1.3 (D): now also Q2.3 (D); no longer Q2.2 (S)
- net at C2.1, R3.1, U1.8 (CE): now also LED1.2 (A), LED2.2 (A); no longer LED1.1 (K), LED2.1 (K)
- net at R2.1: now also LED1.1 (K); no longer LED1.2 (A)
- net at R1.1: now also LED2.1 (K); no longer LED2.2 (A)
- removed net B-: Q2.3 (D), Rprog2.1
- new net: J1.A5 (CC1), J1.B5 (CC2), R4.1
- new net: Q1.1 (G), U2.1 (OD)
- new net: D1.2 (A), J1.A4 (VBUS), J1.A9 (VBUS), J1.B4 (VBUS), J1.B9 (VBUS)
- new net D+: D3.2 (A), J1.A6 (D+), J1.B6 (D+)
- new net D-: D2.2 (A), J1.A7 (D-), J1.B7 (D-)
Other:
- moved on the sheet: Q1, Q2, U2
